File: hardware/v01/electrical/godwit-v01.sch (EAGLE design)
At the start: 85 parts, among them J1 USB-MINIB-M26FTR, U1 BQ24251, U2 LM3668-3034, U3 UC530, U4 AAT4280A, U5 BMP180, U6 MAG3110, U7 ATUCL4U-TQFP48

Commit message: Started ADC input.
Parts:
- added R16, R17: (no value), hybridpi-rcl:R-US_R0603
Connections:
- new net N$46: R16.1, R17.2
- net GND: now also R17.1
- net VBUS: now also R16.2
Changed lines of the file:
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@@
 <layers>
 <layer number="1" name="Top" color="4" fill="1" visible="no" active="no"/>
+<layer number="2" name="Route2" color="1" fill="3" visible="no" active="no"/>
+<layer number="3" name="Route3" color="4" fill="3" visible="no" active="no"/>
+<layer number="4" name="Route4" color="1" fill="4" visible="no" active="no"/>
+<layer number="5" name="Route5" color="4" fill="4" visible="no" active="no"/>
+<layer number="6" name="Route6" color="1" fill="8" visible="no" active="no"/>
+<layer number="7" name="Route7" color="4" fill="8" visible="no" active="no"/>
+<layer number="8" name="Route8" color="1" fill="2" visible="no" active="no"/>
+<layer number="9" name="Route9" color="4" fill="2" visible="no" active="no"/>
+<layer number="10" name="Route10" color="1" fill="7" visible="no" active="no"/>
+<layer number="11" name="Route11" color="4" fill="7" visible="no" active="no"/>
+<layer number="12" name="Route12" color="1" fill="5" visible="no" active="no"/>
+<layer number="13" name="Route13" color="4" fill="5" visible="no" active="no"/>
+<layer number="14" name="Route14" color="1" fill="6" visible="no" active="no"/>
+<layer number="15" name="Route15" color="4" fill="6" visible="no" active="no"/>
 <layer number="16" name="Bottom" color="1" fill="1" visible="no" active="no"/>
 <layer number="17" name="Pads" color="2" fill="1" visible="no" active="no"/>
@@
 <part name="R15" library="hybridpi-rcl" deviceset="R-US_" device="R0603" value="100K"/>
 <part name="SUPPLY9" library="hybridpi-aesthetics" deviceset="3.0V" device=""/>
+<part name="R16" library="hybridpi-rcl" deviceset="R-US_" device="R0603"/>
+<part name="R17" library="hybridpi-rcl" deviceset="R-US_" device="R0603"/>
+<part name="GND26" library="SparkFun-Aesthetics" deviceset="GND" device=""/>
 </parts>
 <sheets>
@@
 <instance part="R15" gate="G$1" x="246.38" y="45.72" rot="R90"/>
 <instance part="SUPPLY9" gate="G$1" x="208.28" y="55.88"/>
+<instance part="R16" gate="G$1" x="297.18" y="116.84" rot="R90"/>
+<instance part="R17" gate="G$1" x="297.18" y="101.6" rot="R90"/>
+<instance part="GND26" gate="1" x="297.18" y="91.44"/>
 </instances>
 <busses>
@@
 <wire x1="236.22" y1="25.4" x2="236.22" y2="22.86" width="0.1524" layer="91"/>
 <junction x="236.22" y="22.86"/>
+</segment>
+<segment>
+<pinref part="R17" gate="G$1" pin="1"/>
+<pinref part="GND26" gate="1" pin="GND"/>
+<wire x1="297.18" y1="96.52" x2="297.18" y2="93.98" width="0.1524" layer="91"/>
 </segment>
 </net>
@@
 <pinref part="R1" gate="G$1" pin="1"/>
 </segment>
+<segment>
+<pinref part="R16" gate="G$1" pin="2"/>
+<wire x1="297.18" y1="121.92" x2="297.18" y2="124.46" width="0.1524" layer="91"/>
+<label x="297.18" y="124.46" size="1.778" layer="95" rot="R90" xref="yes"/>
+</segment>
 </net>
 <net name="CHRG_SCL" class="0">
@@
 </segment>
 </net>
+<net name="N$46" class="0">
+<segment>
+<pinref part="R16" gate="G$1" pin="1"/>
+<pinref part="R17" gate="G$1" pin="2"/>
+<wire x1="297.18" y1="111.76" x2="297.18" y2="106.68" width="0.1524" layer="91"/>
+</segment>
+</net>

Commit message: Finished first draft schematic and layout.
Parts:
- removed R11: 0R, hybridpi-rcl:R-US_R0603
- added C34, C35, C36, C37, C38, C39, C40, C41, C45, C47: 0.1uF, hybridpi-rcl:C-EUC0603
- added C42, C44: 33nF, hybridpi-rcl:C-EUC0603
- added C43: 22uF, hybridpi-rcl:C-EUC0805
- added C46: 2.2uF, hybridpi-rcl:C-EUC0603
- added JP3: M02-JST-PH-2-RA, hybridpi-connector:M02-JST-PH-2-RA
- added JP4: (no value), hybridpi-connector:M03X2NO_SILK
- added L3, L4, L5: 2.5K, hybridpi:FERRITE-BEAD-0603
- added R18, R19, R20, R21, R22: 10K, hybridpi-rcl:R-US_R0603
- added SJ1: SOLDERJUMPERNC, hybridpi-passive:SOLDERJUMPERNC
- added U$18, U$19, U$20: NC, hybridpi-aesthetics:NC
- R1, R10, R3: value 47K -> 100K
- R16: value (none) -> 59K
- R17: value (none) -> 41.2K
- R9: value 470K -> 100K
- S1, S2, S3, S4, S5: device hybridpi-electromechanical:TAC_SWITCHPTH -> hybridpi-electromechanical:TAC_SWITCH-FSMRA; VENDOR (none) -> DIGI-KEY; VENDOR_PN (none) -> 450-1661-ND
Connections:
- new net !RESET!: JP4.1, R22.1, U7.!RESET!
- new net N$47: JP3.1, U7.PA14
- new net N$48: C14.1, L5.1, U5.VDD, U5.VDDIO
- new net N$49: JP3.2, U7.PA20
- new net N$50: C47.1, L4.1, U7.ADVREFP, U7.VDDANA
- new net N$53: C45.1, C46.2, L4.2, U7.VDDCORE
- new net N$54: C15.1, C16.2, L3.1, U6.VDD, U6.VDDIO
- new net N$55: JP4.3, U$18.NC
- new net N$56: JP4.5, U$19.NC
- new net N$57: JP4.4, U$20.NC
- net 3.0V: now also C41.1, C42.1, C43.1, C44.1, JP4.2, L3.2, L5.2, R18.2, R19.2, R20.2, R21.2, R22.2, U7.VDDIN, U7.VDDIO; no longer C14.1, C15.1, C16.2, U5.VDD, U5.VDDIO, U6.VDD, U6.VDDIO
- net 3V_EN: now also U7.PB04
- net B_BCK: now also C38.1, S5.2; no longer S5.3, S5.4
- net B_DWN: now also C37.1, S4.2; no longer S4.3, S4.4
- net B_SEL: now also C36.1, S3.2; no longer S3.3, S3.4
- net B_UP: now also C35.1, S2.2; no longer S2.3, S2.4
- net CHRG_SCL: now also R19.1
- net CHRG_SDA: now also R18.1
- net GND: now also C34.2, C35.2, C36.2, C37.2, C38.2, C39.1, C40.2, C41.2, C42.2, C43.2, C44.2, C45.2, C46.1, C47.2, JP4.6, U7.GND, U7.GNDANA; no longer S2.2, S3.2, S4.2, S5.2
- net N$35: now also SJ1.2; no longer R11.1
- net N$42: now also SJ1.1; no longer R11.2
- net N$46: now also C40.1, U7.PA19
- net N$9: now also C34.1
- net PWR_TACT: no longer S1.2
- net SD_CRD_DET: now also C39.2, U7.PA11
- net SENS_SCL: now also R21.1
- net SENS_SDA: now also R20.1
- net VBUS: no longer R16.2
- net VSYS: now also R16.2, S1.2; no longer S1.3, S1.4
Other:
- moved on the sheet: D2, D3, R1, R12, R13, R14, R15, R16, R17, R2, R3, U7
