File: hardware/v01/electrical/godwit-v01.sch (EAGLE design)
At the start: 114 parts, among them J1 USB-MINIB-M26FTR, U1 BQ24251, U2 LM3668-3034, U3 UC530, U4 AAT4280A, U5 BMP180, U6 MAG3110, U7 ATUCL4U-TQFP48

Commit message: Added current limiting resistors and finalized v01 design.
Parts:
- added R11, R23: 100K, hybridpi-rcl:R-US_R0603
Connections:
- net !PG! renamed !PG!_LED
- new net N$88: R11.1, R2.2, R3.2, S1.1
- new net STAT_LED: D1.CR, R23.2, U1.STAT
- net CHRG_STAT: now also R23.1; no longer D1.CR, U1.STAT
- net PWR_TACT: now also R11.2; no longer R2.2, R3.2, S1.1
Other:
- note added: "1.0"
- note added: "1002"
- note added: "ADG"
Changed lines of the file:
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@@
 <setting verticaltext="up"/>
 </settings>
-<grid distance="0.1" unitdist="inch" unit="inch" style="lines" multiple="1" display="no" altdistance="0.01" altunitdist="inch" altunit="inch"/>
+<grid distance="0.1" unitdist="inch" unit="inch" style="lines" multiple="1" display="yes" altdistance="0.01" altunitdist="inch" altunit="inch"/>
 <layers>
 <layer number="1" name="Top" color="4" fill="1" visible="no" active="no"/>
@@
 <part name="SUPPLY15" library="hybridpi-aesthetics" deviceset="3.0V" device=""/>
 <part name="SJ1" library="hybridpi-passive" deviceset="SOLDERJUMPER" device="NC"/>
+<part name="R11" library="hybridpi-rcl" deviceset="R-US_" device="R0603" value="100K"/>
+<part name="R23" library="hybridpi-rcl" deviceset="R-US_" device="R0603" value="100K"/>
 </parts>
 <sheets>
 <sheet>
 <plain>
+<text x="398.78" y="20.32" size="2.54" layer="94" align="center-left">ADG</text>
+<text x="363.22" y="12.7" size="2.54" layer="94" align="center-left">1002</text>
+<text x="416.56" y="7.62" size="2.54" layer="94">1.0</text>
 </plain>
 <instances>
@@
 <attribute name="NAME" x="53.848" y="95.25" size="1.778" layer="95"/>
 </instance>
+<instance part="R11" gate="G$1" x="154.94" y="203.2" rot="R180"/>
+<instance part="R23" gate="G$1" x="93.98" y="210.82" rot="R180"/>
 </instances>
 <busses>
@@
 <wire x1="91.44" y1="236.22" x2="78.74" y2="236.22" width="0.1524" layer="91"/>
 <wire x1="78.74" y1="236.22" x2="78.74" y2="203.2" width="0.1524" layer="91"/>
-<wire x1="78.74" y1="203.2" x2="93.98" y2="203.2" width="0.1524" layer="91"/>
-<label x="93.98" y="203.2" size="1.27" layer="95" xref="yes"/>
+<wire x1="78.74" y1="203.2" x2="101.6" y2="203.2" width="0.1524" layer="91"/>
+<label x="101.6" y="203.2" size="1.27" layer="95" xref="yes"/>
 </segment>
 <segment>
@@
 <wire x1="91.44" y1="233.68" x2="81.28" y2="233.68" width="0.1524" layer="91"/>
 <wire x1="81.28" y1="233.68" x2="81.28" y2="205.74" width="0.1524" layer="91"/>
-<wire x1="81.28" y1="205.74" x2="93.98" y2="205.74" width="0.1524" layer="91"/>
-<label x="93.98" y="205.74" size="1.27" layer="95" xref="yes"/>
+<wire x1="81.28" y1="205.74" x2="101.6" y2="205.74" width="0.1524" layer="91"/>
+<label x="101.6" y="205.74" size="1.27" layer="95" xref="yes"/>
 </segment>
 <segment>
@@
 </segment>
 </net>
-<net name="!PG!" class="0">
+<net name="!PG!_LED" class="0">
 <segment>
 <pinref part="U1" gate="G$1" pin="!PG!"/>
@@
 </segment>
 </net>
-<net name="CHRG_STAT" class="0">
+<net name="STAT_LED" class="0">
 <segment>
 <pinref part="U1" gate="G$1" pin="STAT"/>
@@
 <wire x1="53.34" y1="213.36" x2="53.34" y2="210.82" width="0.1524" layer="91"/>
 <wire x1="53.34" y1="210.82" x2="86.36" y2="210.82" width="0.1524" layer="91"/>
-<wire x1="86.36" y1="210.82" x2="93.98" y2="210.82" width="0.1524" layer="91"/>
+<pinref part="R23" gate="G$1" pin="2"/>
+<wire x1="88.9" y1="210.82" x2="86.36" y2="210.82" width="0.1524" layer="91"/>
 <junction x="86.36" y="210.82"/>
-<label x="93.98" y="210.82" size="1.27" layer="95" xref="yes"/>
 <label x="55.88" y="210.82" size="1.778" layer="95"/>
-</segment>
-<segment>
-<pinref part="U7" gate="G$1" pin="PA13"/>
-<wire x1="218.44" y1="96.52" x2="220.98" y2="96.52" width="0.1524" layer="91"/>
-<label x="220.98" y="96.52" size="1.27" layer="95" xref="yes"/>
 </segment>
 </net>
@@
 <net name="PWR_TACT" class="0">
 <segment>
-<pinref part="R2" gate="G$1" pin="2"/>
-<wire x1="162.56" y1="208.28" x2="162.56" y2="203.2" width="0.1524" layer="91"/>
-<pinref part="R3" gate="G$1" pin="2"/>
-<wire x1="162.56" y1="203.2" x2="162.56" y2="200.66" width="0.1524" layer="91"/>
-<wire x1="162.56" y1="200.66" x2="162.56" y2="198.12" width="0.1524" layer="91"/>
-<wire x1="165.1" y1="200.66" x2="162.56" y2="200.66" width="0.1524" layer="91"/>
-<junction x="162.56" y="200.66"/>
-<wire x1="162.56" y1="203.2" x2="157.48" y2="203.2" width="0.1524" layer="91"/>
-<junction x="162.56" y="203.2"/>
-<label x="157.48" y="203.2" size="1.27" layer="95" rot="R180" xref="yes"/>
-<pinref part="S1" gate="S" pin="1"/>
-</segment>
-<segment>
 <pinref part="U7" gate="G$1" pin="PB10"/>
 <wire x1="180.34" y1="76.2" x2="177.8" y2="76.2" width="0.1524" layer="91"/>
 <label x="177.8" y="76.2" size="1.27" layer="95" rot="R180" xref="yes"/>
+</segment>
+<segment>
+<pinref part="R11" gate="G$1" pin="2"/>
+<wire x1="149.86" y1="203.2" x2="147.32" y2="203.2" width="0.1524" layer="91"/>
+<label x="147.32" y="203.2" size="1.27" layer="95" rot="R180" xref="yes"/>
 </segment>
 </net>
@@
 </segment>
 </net>
+<net name="N$88" class="0">
+<segment>
+<pinref part="R2" gate="G$1" pin="2"/>
+<wire x1="162.56" y1="208.28" x2="162.56" y2="203.2" width="0.1524" layer="91"/>
+<pinref part="R3" gate="G$1" pin="2"/>
+<wire x1="162.56" y1="203.2" x2="162.56" y2="200.66" width="0.1524" layer="91"/>
+<wire x1="162.56" y1="200.66" x2="162.56" y2="198.12" width="0.1524" layer="91"/>
+<wire x1="165.1" y1="200.66" x2="162.56" y2="200.66" width="0.1524" layer="91"/>
+<junction x="162.56" y="200.66"/>
+<pinref part="S1" gate="S" pin="1"/>
+<pinref part="R11" gate="G$1" pin="1"/>
+<wire x1="160.02" y1="203.2" x2="162.56" y2="203.2" width="0.1524" layer="91"/>
+<junction x="162.56" y="203.2"/>
+</segment>
+</net>
+<net name="CHRG_STAT" class="0">
+<segment>
+<pinref part="R23" gate="G$1" pin="1"/>
+<wire x1="99.06" y1="210.82" x2="101.6" y2="210.82" width="0.1524" layer="91"/>
+<label x="101.6" y="210.82" size="1.27" layer="95" xref="yes"/>
+</segment>
+<segment>
+<pinref part="U7" gate="G$1" pin="PA13"/>
+<wire x1="218.44" y1="96.52" x2="220.98" y2="96.52" width="0.1524" layer="91"/>
+<label x="220.98" y="96.52" size="1.27" layer="95" xref="yes"/>
+</segment>
+</net>

Commit message: Started to add BOM.
Parts:
- removed J1: USB-MINIB-M26FTR, hybridpi-connector:USB-MINIB-M26FTR
- removed U$15: 128240D, hybridpi-connector:128240D
- added JP5: (no value), hybridpi-connector:M03X2NO_SILK
- added JP6: M02-JST-PH-2-RA, hybridpi-connector:M02-JST-PH-2-RA
- C1: value 10uF -> 1uF; device hybridpi-rcl:C-EUC0805 -> hybridpi-rcl:C-EUC0603; VENDOR_PN 490-6470-1-ND -> 587-1248-1-ND
- C10, C12, C16, C8: VENDOR (none) -> DIGI-KEY; VENDOR_PN (none) -> 587-1248-1-ND; VOLTAGE >=10V -> (none)
- C11: value 2.2uF -> 1uF; VENDOR DIGI-KEY -> (none); VENDOR_PN 445-5167-1-ND -> (none); VOLTAGE (none) -> >=10V
- C13: value 4.7uF -> 10uF; device hybridpi-rcl:C-EUC0603 -> hybridpi-rcl:C-EUC0805; VENDOR_PN 490-3297-1-ND -> 490-6470-1-ND; VOLTAGE >=10V -> (none)
- C14: value 0.1uF -> DNP; VENDOR (none) -> DIGI-KEY; VENDOR_PN (none) -> 587-1248-1-ND
- C15, C17, C18, C2, C4: value 0.1uF -> 1uF; VENDOR (none) -> DIGI-KEY; VENDOR_PN (none) -> 587-1248-1-ND
- C19: value 10uF -> 33nF; device hybridpi-rcl:C-EUC0805 -> hybridpi-rcl:C-EUC0603; VENDOR DIGI-KEY -> (none); VENDOR_PN 490-6470-1-ND -> (none); VOLTAGE (none) -> >15
- C20, C38, C40: value 0.1uF -> 1uF; VOLTAGE (none) -> >=10V
- C21, C28: value 1uF -> 22uF; device hybridpi-rcl:C-EUC0603 -> hybridpi-rcl:C-EUC0805; VENDOR_PN 587-1248-1-ND -> 587-1305-1-ND
- C22, C27: value 1uF -> 2.2uF; VENDOR_PN 587-1248-1-ND -> 445-5167-1-ND
- C23: value DNP -> 0.1uF; VENDOR DIGI-KEY -> (none); VENDOR_PN 587-1248-1-ND -> (none)
- C24, C25, C30, C32, C33: value 1uF -> 0.1uF; VENDOR DIGI-KEY -> (none); VENDOR_PN 587-1248-1-ND -> (none)
- C26, C29: value 1uF -> 33nF; VENDOR DIGI-KEY -> (none); VENDOR_PN 587-1248-1-ND -> (none)
- C3, C43, C6: value 22uF -> 0.1uF; device hybridpi-rcl:C-EUC0805 -> hybridpi-rcl:C-EUC0603; VENDOR DIGI-KEY -> (none); VENDOR_PN 587-1305-1-ND -> (none)
- C31: value 1uF -> 10uF; device hybridpi-rcl:C-EUC0603 -> hybridpi-rcl:C-EUC0805; VENDOR_PN 587-1248-1-ND -> 490-6470-1-ND
- C35: value 0.1uF -> 22uF; device hybridpi-rcl:C-EUC0603 -> hybridpi-rcl:C-EUC0805; VENDOR (none) -> DIGI-KEY; VENDOR_PN (none) -> 587-1305-1-ND
- C37: value 0.1uF -> 4.7uF; VENDOR (none) -> DIGI-KEY; VENDOR_PN (none) -> 490-3297-1-ND; VOLTAGE (none) -> >=10V
- C42, C44: value 33nF -> 0.1uF
- C46: value 2.2uF -> 0.1uF; VENDOR DIGI-KEY -> (none); VENDOR_PN 445-5167-1-ND -> (none)
- C5: value 33nF -> 1uF; VENDOR (none) -> DIGI-KEY; VENDOR_PN (none) -> 587-1248-1-ND; VOLTAGE >15 -> (none)
- C7: value 0.1uF -> 2.2uF; VENDOR (none) -> DIGI-KEY; VENDOR_PN (none) -> 445-5167-1-ND
- C9: value 2.2uF -> 1uF; VENDOR_PN 445-5167-1-ND -> 587-1248-1-ND
- D2, D3: value (none) -> 1N4148X-TP; VENDOR (none) -> DIGI-KEY; VENDOR_PN (none) -> 1N4148XTPMSCT-ND
- JP3: value M02-JST-PH-2-RA -> USB-MINIB-M26FTR; device hybridpi-connector:M02-JST-PH-2-RA -> hybridpi-connector:USB-MINIB-M26FTR
- JP4: value (none) -> 128240D; device hybridpi-connector:M03X2NO_SILK -> hybridpi-connector:128240D
- L1: value 2.2uH -> 1uH
- L2: value 1uH -> 2.5K; device hybridpi:INDUCTOR-SRU5028 -> hybridpi:FERRITE-BEAD-0603; VENDOR (none) -> DIGI-KEY; VENDOR_PN (none) -> 587-1893-1-ND
- L3: value 2.5K -> 2.2uH; device hybridpi:FERRITE-BEAD-0603 -> hybridpi:INDUCTOR-SRU5028; VENDOR DIGI-KEY -> (none); VENDOR_PN 587-1893-1-ND -> (none)
- R1, R3: value 100K -> 2.2K
- R10, R11, R12, R13: value 100K -> 10K
- R14: value 100K -> 59K
- R15: value 100K -> 41.2K
- R16: value 59K -> 100K
- R17: value 41.2K -> 100K
- R18, R20: value 10K -> 100K
- R19, R21, R22: value 10K -> 220R
- R2, R5: value 2.2K -> 100K
- R4, R8: value 220R -> 100K
- R6: value 2.2K -> 10K
- R7: value 220R -> 2.2K
- S1, S2, S3, S4, S5: value (none) -> FSMRA7JH
- U2: value LM3668-3034 -> ATUCL4U-TQFP48; device hybridpi:LM3668-3034 -> hybridpi-digitalic:ATUCL4U-TQFP48
- U3: value UC530 -> LM3668-3034; device hybridpi-rf:UC530 -> hybridpi:LM3668-3034
- U5: value BMP180 -> UC530; device hybridpi-sensor:BMP180 -> hybridpi-rf:UC530
- U6: value MAG3110 -> BMP180; device hybridpi-sensor:MAG3110 -> hybridpi-sensor:BMP180
- U7: value ATUCL4U-TQFP48 -> MAG3110; device hybridpi-digitalic:ATUCL4U-TQFP48 -> hybridpi-sensor:MAG3110
- renumbered U$1 to U$80
Connections:
- net !RESET!: now also JP5.1, R10.1, U2.!RESET!; no longer JP4.1, R22.1, U7.!RESET!
- net 3.0V: now also C13.2, C21.1, C24.1, C26.1, C29.1, C34.1, C35.1, C4.2, C6.2, JP4.IF1, JP4.IF2, JP4.VDD, JP5.2, L4.2, R10.2, R11.2, R16.2, R17.2, R2.1, R23.2, R6.2, U2.VDDIN, U2.VDDIO, U3.FB, U3.VOUT; no longer C19.2, C20.2, C3.1, C33.2, C4.1, C41.1, C42.1, C43.1, C44.1, JP4.2, L3.2, R10.1, R14.2, R15.2, R19.2, R21.2, R22.2, R9.2, U$15.IF1, U$15.IF2, U$15.VDD, U2.FB, U2.VOUT, U7.VDDIN, U7.VDDIO
- net 3V_EN: now also D3.A, U2.PB04; no longer D2.A, U7.PB04
- net B_BCK: now also C47.1, R23.1, U2.PB09; no longer C38.1, R15.1, U7.PB09
- net B_DWN: now also C46.1, R20.1, U2.PB08; no longer C37.1, R14.1, U7.PB08
- net B_SEL: now also C42.1, R18.1, U2.PA15; no longer C36.1, R13.1, U7.PA15
- net B_UP: now also C39.1, R17.1, U2.PA16; no longer C35.1, R12.1, U7.PA16
- net CHRG_SCL: now also R13.1, U2.PA04; no longer R19.1, U7.PA04
- net CHRG_SDA: now also R12.1, U2.PA17; no longer R18.1, U7.PA17
- net CHRG_STAT: now also R4.1, U2.PA13; no longer R23.1, U7.PA13
- net GND: now also C12.2, C20.2, C21.2, C22.1, C23.2, C24.2, C25.2, C26.2, C27.1, C3.1, C33.2, C37.1, C38.1, C39.2, C4.1, C40.1, C46.2, C5.2, C6.1, C7.1, JP3.GND, JP4.IF3, JP4.SHIELD, JP4.VSS, JP5.6, R15.1, R7.1, U2.GNDANA, U3.SYNC/MODE, U3.VSEL; no longer C10.1, C12.1, C14.2, C16.1, C17.2, C18.2, C19.1, C20.1, C27.2, C3.2, C33.1, C37.2, C38.2, C39.1, C4.2, C40.2, C46.1, C6.2, C7.2, C9.1, J1.GND, JP4.6, R17.1, R2.1, U$15.IF3, U$15.SHIELD, U$15.VSS, U2.SYNC/MODE, U2.VSEL, U7.GNDANA
- net GPS_RX: now also R22.2, U2.PB06; no longer R7.2, U7.PB06
- net GPS_TX: now also R21.2, U2.PB07; no longer R4.2, U7.PB07
- net LCD_!CS!: now also JP4.XCS, U2.PA01; no longer U$15.XCS, U7.PA01
- net LCD_!RST!: now also JP4.RST, U2.PA02; no longer U$15.RST, U7.PA02
- net LCD_A0: now also JP4.A0, U2.PA18; no longer U$15.A0, U7.PA18
- net LCD_D0: now also JP4.D0, U2.PA10; no longer U$15.D0, U7.PA10
- net LCD_D1: now also JP4.D1, U2.PA12; no longer U$15.D1, U7.PA12
- net LCD_D2: now also JP4.D2, U2.PA09; no longer U$15.D2, U7.PA09
- net LCD_D3: now also JP4.D3, U2.PA08; no longer U$15.D3, U7.PA08
- net LCD_D4: now also JP4.D4, U2.PA03; no longer U$15.D4, U7.PA03
- net LCD_D5: now also JP4.D5, U2.PB12; no longer U$15.D5, U7.PB12
- net LCD_D6: now also JP4.D6, U2.PA22; no longer U$15.D6, U7.PA22
- net LCD_D7: now also JP4.D7, U2.PA00; no longer U$15.D7, U7.PA00
- net LCD_RD: now also JP4.E_RD, U2.PA05; no longer U$15.E_RD, U7.PA05
- net LCD_WR: now also JP4.RW/WR, U2.PB11; no longer U$15.RW/WR, U7.PB11
- net LDO: now also C11.2; no longer C10.2
- net N$1: now also L3.2, U3.SW2; no longer L1.2, U2.SW2
- net N$10: now also U5.TX1; no longer U3.TX1
- net N$11: now also U5.RX1; no longer U3.RX1
- net N$12: now also U5.PPS; no longer U3.PPS
- net N$13: now also U5.EINT1; no longer U3.EINT1
- net N$14: now also U5.32K/DR_INT; no longer U3.32K/DR_INT
- net N$15: now also R1.1; no longer R5.1
- net N$16: now also U5.GPIO9; no longer U3.GPIO9
- net N$17: now also U5.GPIO10; no longer U3.GPIO10
- net N$18: now also R3.1; no longer R6.1
- net N$19: now also U5.WAKEUP; no longer U3.WAKEUP
- net N$2: now also L3.1, U3.SW1; no longer L1.1, U2.SW1
- net N$20: now also U5.UI_FIX; no longer U3.UI_FIX
- net N$21: now also U5.!RESET!; no longer U3.!RESET!
- net N$22: now also C37.2, U5.VDD; no longer C13.2, U3.VDD
- net N$23: now also R21.1, U5.TX0; no longer R4.1, U3.TX0
- net N$24: now also R22.1, U5.RX0; no longer R7.1, U3.RX0
- net N$25: now also R19.2, U5.TIMER; no longer R8.2, U3.TIMER
- net N$26: now also R16.1, R19.1; no longer R8.1, R9.1
- net N$27: now also C10.1, C14.1, C9.2, JP4.C2N; no longer C21.2, C22.1, C23.1, U$15.C2N
- net N$28: now also C44.1, U7.CAP-R; no longer C18.1, U6.CAP-R
- net N$29: now also C43.1, U7.CAP-A; no longer C17.1, U6.CAP-A
- net N$3: now also C19.1; no longer C5.1
- net N$32: now also U7.INT1; no longer U6.INT1
- net N$33: now also C9.1, JP4.C2P; no longer C21.1, U$15.C2P
- net N$34: now also C10.2, JP4.C4P; no longer C22.2, U$15.C4P
- net N$35: now also C14.2, JP4.C6P; no longer C23.2, U$15.C6P
- net N$36: now also C16.1, C17.2, C18.1, JP4.C1N; no longer C24.2, C25.1, C26.1, U$15.C1N
- net N$37: now also C17.1, JP4.C1P; no longer C24.1, U$15.C1P
- net N$38: now also C16.2, JP4.C3P; no longer C25.2, U$15.C3P
- net N$39: now also C18.2, JP4.C5P; no longer C26.2, U$15.C5P
- net N$4: now also U5.ANT, U5.RF_IN; no longer U3.ANT, U3.RF_IN
- net N$40: now also C2.1, JP4.V4; no longer C28.1, U$15.V4
- net N$41: now also C5.1, JP4.V3; no longer C29.1, U$15.V3
- net N$42: now also C1.1, JP4.C7P, JP4.VLCD; no longer C27.1, U$15.C7P, U$15.VLCD
- net N$43: now also C8.1, JP4.V2; no longer C30.1, U$15.V2
- net N$44: now also C12.1, JP4.V1; no longer C31.1, U$15.V1
- net N$45: now also C15.1, JP4.V0IN, JP4.V0OUT; no longer C32.1, U$15.V0IN, U$15.V0OUT
- net N$46: now also C36.1, R14.1, R15.2, U2.PA19; no longer C40.1, R16.1, R17.2, U7.PA19
- net N$47: now also JP6.1, U2.PA14; no longer JP3.1, U7.PA14
- net N$48: now also C45.1, U6.VDD, U6.VDDIO; no longer C14.1, U5.VDD, U5.VDDIO
- net N$49: now also JP6.2, U2.PA20; no longer JP3.2, U7.PA20
- net N$5: now also C19.2, L1.1; no longer C5.2, L2.1
- net N$50: now also C23.1, L2.1, U2.ADVREFP, U2.VDDANA; no longer C47.1, L4.1, U7.ADVREFP, U7.VDDANA
- net N$51: now also JP4.SCL; no longer U$15.SCL
- net N$52: now also JP4.SI; no longer U$15.SI
- net N$53: now also C27.2, C30.1, L2.2, U2.VDDCORE; no longer C45.1, C46.2, L4.2, U7.VDDCORE
- net N$54: now also C40.2, C41.1, L4.1, U7.VDD, U7.VDDIO; no longer C15.1, C16.2, L3.1, U6.VDD, U6.VDDIO
- net N$55: now also JP5.3; no longer JP4.3
- net N$56: now also JP5.5; no longer JP4.5
- net N$57: now also JP5.4; no longer JP4.4
- net N$6: now also C20.1; no longer C8.1
- net N$8: now also D2.A, R9.2; no longer D3.A, R1.2
- net N$88: now also R5.1, R7.2, R8.2; no longer R11.1, R2.2, R3.2
- net N$9: now also C32.1, R8.1, U3.EN; no longer C34.1, R3.1, U2.EN
- net PWR_TACT: now also R5.2, U2.PB10; no longer R11.2, U7.PB10
- net SD_!CS!: now also U2.PB00; no longer U7.PB00
- net SD_CRD_DET: now also C3.2, R2.2, U2.PA11; no longer C39.2, R10.2, U7.PA11
- net SD_MISO: now also U2.PB02; no longer U7.PB02
- net SD_MOSI: now also U2.PB03; no longer U7.PB03
- net SD_SCLK: now also U2.PA06; no longer U7.PA06
- net SENS_SCL: now also R6.1, U2.PB05, U7.SCL; no longer R21.1, U5.SCL, U7.PB05
- net SENS_SDA: now also R11.1, U2.PA21, U7.SDA; no longer R20.1, U5.SDA, U7.PA21
- net STAT_LED: now also R4.2; no longer R23.2
- net USB_D+: now also JP3.D+, U2.PB14; no longer J1.D+, U7.PB14
- net USB_D-: now also JP3.D-, U2.PB13; no longer J1.D-, U7.PB13
- net VBUS: now also C7.2, JP3.VBUS, R9.1; no longer C9.2, J1.VBUS, R1.1
- net VSYS: now also C25.1, C28.1, C31.1, C33.1, C38.2, L1.2, R1.2, R14.2, R3.2, U3.VDD, U3.VIN, U5.VDD_B; no longer C1.1, C12.2, C2.1, C6.1, C7.1, L2.2, R16.2, R5.2, R6.2, U2.VDD, U2.VIN, U3.VDD_B
- net V_BATT: now also C22.2; no longer C11.2
Other:
- moved on the sheet: C1, C10, C11, C12, C13, C14, C15, C16, C17, C18, C19, C2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

Commit message: Finished BOM
Parts:
- L1: value 1uH -> 1.2uH
- U2: value ATUCL4U-TQFP48 -> ATUC128L4U-TQFP48; device hybridpi-digitalic:ATUCL4U-TQFP48 -> hybridpi-digitalic:ATUC128L4U-TQFP48
Changed lines of the file:
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@@
 <setting verticaltext="up"/>
 </settings>
-<grid distance="0.1" unitdist="inch" unit="inch" style="lines" multiple="1" display="yes" altdistance="0.01" altunitdist="inch" altunit="inch"/>
+<grid distance="0.1" unitdist="inch" unit="inch" style="lines" multiple="1" display="no" altdistance="0.01" altunitdist="inch" altunit="inch"/>
 <layers>
 <layer number="1" name="Top" color="4" fill="1" visible="no" active="no"/>
@@
 <parts>
 <part name="L3" library="hybridpi" deviceset="INDUCTOR" device="-SRU5028" value="2.2uH"/>
-<part name="L1" library="hybridpi" deviceset="INDUCTOR" device="-SRU5028" value="1uH"/>
+<part name="L1" library="hybridpi" deviceset="INDUCTOR" device="-SRU5028" value="1.2uH"/>
 <part name="U1" library="hybridpi" deviceset="BQ24251" device=""/>
 <part name="U3" library="hybridpi" deviceset="LM3668" device="-3034"/>
@@
 <part name="SUPPLY8" library="hybridpi-aesthetics" deviceset="3.0V" device=""/>
 <part name="GND24" library="SparkFun-Aesthetics" deviceset="GND" device=""/>
-<part name="U2" library="hybridpi-digitalic" deviceset="ATUC*L" device="4U-TQFP48"/>
+<part name="U2" library="hybridpi-digitalic" deviceset="ATUC*L" device="4U-TQFP48" technology="128"/>
 <part name="GND25" library="SparkFun-Aesthetics" deviceset="GND" device=""/>
 <part name="R17" library="hybridpi-rcl" deviceset="R-US_" device="R0603" value="100K"/>
