File: hardware/v01/electrical/godwit-v01.brd (EAGLE design)
At the start: 72.5 x 132.8 mm, 98 parts, among them J1 USB-MINIB-M26FTR, U1 BQ24251, U2 LM3668-3034, U3 UC530, U4 AAT4280A, U5 BMP180, U6 MAG3110, U7 ATUCL4U-TQFP48

Commit message: Started to add BOM.
Parts:
- removed J1: USB-MINIB-M26FTR, hybridpi-connector:USB-MINIB-M26FTR
- removed U$15: 128240D, hybridpi-connector:128240D
- added JP5: (no value), hybridpi-connector:2X3-NS
- added JP6: M02-JST-PH-2-RA, hybridpi-connector:JST-PH-2-RA
- C1: value 10uF -> 1uF; device hybridpi-rcl:C0805 -> hybridpi-rcl:C0603
- C11, C9: value 2.2uF -> 1uF
- C13: value 4.7uF -> 10uF; device hybridpi-rcl:C0603 -> hybridpi-rcl:C0805
- C14: value 0.1uF -> DNP
- C15, C17, C18, C2, C20, C38, C4, C40: value 0.1uF -> 1uF
- C19: value 10uF -> 33nF; device hybridpi-rcl:C0805 -> hybridpi-rcl:C0603
- C21, C28: value 1uF -> 22uF; device hybridpi-rcl:C0603 -> hybridpi-rcl:C0805
- C22, C27: value 1uF -> 2.2uF
- C23: value DNP -> 0.1uF
- C24, C25, C30, C32, C33: value 1uF -> 0.1uF
- C26, C29: value 1uF -> 33nF
- C3, C43, C6: value 22uF -> 0.1uF; device hybridpi-rcl:C0805 -> hybridpi-rcl:C0603
- C31: value 1uF -> 10uF; device hybridpi-rcl:C0603 -> hybridpi-rcl:C0805
- C35: value 0.1uF -> 22uF; device hybridpi-rcl:C0603 -> hybridpi-rcl:C0805
- C37: value 0.1uF -> 4.7uF
- C42, C44: value 33nF -> 0.1uF
- C46: value 2.2uF -> 0.1uF
- C5: value 33nF -> 1uF
- C7: value 0.1uF -> 2.2uF
- D2, D3: value (none) -> 1N4148X-TP
- JP3: value M02-JST-PH-2-RA -> USB-MINIB-M26FTR; device hybridpi-connector:JST-PH-2-RA -> hybridpi-connector:USB-MINIB-M26FTR
- JP4: value (none) -> 128240D; device hybridpi-connector:2X3-NS -> hybridpi-connector:128240D
- L1: value 2.2uH -> 1uH
- L2: value 1uH -> 2.5K; device hybridpi:SRU5028 -> hybridpi:0603
- L3: value 2.5K -> 2.2uH; device hybridpi:0603 -> hybridpi:SRU5028
- R1, R3: value 100K -> 2.2K
- R10, R11, R12, R13: value 100K -> 10K
- R14: value 100K -> 59K
- R15: value 100K -> 41.2K
- R16: value 59K -> 100K
- R17: value 41.2K -> 100K
- R18, R20: value 10K -> 100K
- R19, R21, R22: value 10K -> 220R
- R2, R5: value 2.2K -> 100K
- R4, R8: value 220R -> 100K
- R6: value 2.2K -> 10K
- R7: value 220R -> 2.2K
- S1, S2, S3, S4, S5: value (none) -> FSMRA7JH
- U2: value LM3668-3034 -> ATUCL4U-TQFP48; device hybridpi:WSON-12 -> hybridpi-digitalic:TQFP48
- U3: value UC530 -> LM3668-3034; device hybridpi-rf:UC530 -> hybridpi:WSON-12
- U5: value BMP180 -> UC530; device hybridpi-sensor:BMP180 -> hybridpi-rf:UC530
- U6: value MAG3110 -> BMP180; device hybridpi-sensor:DFN-10-2X2 -> hybridpi-sensor:BMP180
- U7: value ATUCL4U-TQFP48 -> MAG3110; device hybridpi-digitalic:TQFP48 -> hybridpi-sensor:DFN-10-2X2
- moved U3 102.0 mm to (16.2, 107.0), turned to 90 degrees
- moved C38 98.8 mm to (28.5, 7.00), turned to 0 degrees
- moved C12 93.0 mm to (19.0, 99.5), turned to 180 degrees
- moved R8 92.2 mm to (12.4, 104.5)
- moved R4 91.3 mm to (7.20, 97.0)
- moved R7 91.1 mm to (12.4, 103.0), turned to 180 degrees
- moved C37 91.1 mm to (28.5, 5.00), turned to 0 degrees
- moved R19 89.3 mm to (38.0, 16.0), turned to 180 degrees
- moved R6 76.2 mm to (21.0, 47.5)
- moved R9 65.3 mm to (7.45, 105.8), turned to 90 degrees
- moved C6 63.4 mm to (15.5, 59.0), turned to 270 degrees
- moved R22 62.3 mm to (41.0, 16.5)
- moved L3 60.7 mm to (21.6, 105.2), turned to 270 degrees
- moved C19 58.3 mm to (15.1, 117.3), turned to 90 degrees
- moved C15 57.5 mm to (18.5, 101.0)
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Connections:
- net !RESET!: now also JP5.1, R10.1, U2.22; no longer JP4.1, R22.1, U7.22
- net 3.0V: now also C13.2, C21.1, C24.1, C26.1, C29.1, C34.1, C35.1, C4.2, C6.2, JP4.13, JP4.14, JP4.20, JP5.2, L4.2, R10.2, R11.2, R16.2, R17.2, R2.1, R23.2, R6.2, U2.17, U2.42, U2.48, U3.1, U3.12; no longer C19.2, C20.2, C3.1, C33.2, C4.1, C41.1, C42.1, C43.1, C44.1, JP4.2, L3.2, R10.1, R14.2, R15.2, R19.2, R21.2, R22.2, R9.2, U$15.13, U$15.14, U$15.20, U2.1, U2.12, U7.17, U7.42, U7.48
- net 3V_EN: now also D3.A, U2.21; no longer D2.A, U7.21
- net B_BCK: now also C47.1, R23.1, U2.29; no longer C38.1, R15.1, U7.29
- net B_DWN: now also C46.1, R20.1, U2.32; no longer C37.1, R14.1, U7.32
- net B_SEL: now also C42.1, R18.1, U2.37; no longer C36.1, R13.1, U7.37
- net B_UP: now also C39.1, R17.1, U2.38; no longer C35.1, R12.1, U7.38
- net CHRG_SCL: now also R13.1, U2.28; no longer R19.1, U7.28
- net CHRG_SDA: now also R12.1, U2.39; no longer R18.1, U7.39
- net CHRG_STAT: now also R4.1, U2.26; no longer R23.1, U7.26
- net GND: now also C12.2, C20.2, C21.2, C22.1, C23.2, C24.2, C25.2, C26.2, C27.1, C3.1, C33.2, C37.1, C38.1, C39.2, C4.1, C40.1, C46.2, C5.2, C6.1, C7.1, JP3.5, JP4.15, JP4.19, JP4.SHIELD1, JP4.SHIELD2, JP5.6, R15.1, R7.1, U2.1, U2.19, U2.33, U2.43, U2.45, U3.3, U3.8, U3.9, U3.PAD, U5.10, U5.11, U5.12, U5.13, U5.14, U5.15, U5.18, U5.19, U5.21, U5.22, U5.27, U5.31, U5.4, U5.5, U6.7, U7.10, U7.5; no longer C10.1, C12.1, C14.2, C16.1, C17.2, C18.2, C19.1, C20.1, C27.2, C3.2, C33.1, C37.2, C38.2, C39.1, C4.2, C40.2, C46.1, C6.2, C7.2, C9.1, J1.5, JP4.6, R17.1, R2.1, U$15.15, U$15.19, U$15.SHIELD1, U$15.SHIELD2, U2.10, U2.11, U2.3, U2.8, U2.9, U2.PAD, U3.12, U3.13, U3.14, U3.15, U3.18, U3.19, U3.21, U3.22, U3.27, U3.31, U3.4, U3.5, U5.7, U6.10, U6.5, U7.1, U7.19, U7.33, U7.43, U7.45
- net GPS_RX: now also R22.2, U2.30; no longer R7.2, U7.30
- net GPS_TX: now also R21.2, U2.31; no longer R4.2, U7.31
- net LCD_!CS!: now also JP4.18, U2.14; no longer U$15.18, U7.14
- net LCD_!RST!: now also JP4.12, U2.13; no longer U$15.12, U7.13
- net LCD_A0: now also JP4.1, U2.41; no longer U$15.1, U7.41
- net LCD_D0: now also JP4.3, U2.46; no longer U$15.3, U7.46
- net LCD_D1: now also JP4.4, U2.47; no longer U$15.4, U7.47
- net LCD_D2: now also JP4.5, U2.2; no longer U$15.5, U7.2
- net LCD_D3: now also JP4.6, U2.3; no longer U$15.6, U7.3
- net LCD_D4: now also JP4.7, U2.4; no longer U$15.7, U7.4
- net LCD_D5: now also JP4.8, U2.5; no longer U$15.8, U7.5
- net LCD_D6: now also JP4.9, U2.9; no longer U$15.9, U7.9
- net LCD_D7: now also JP4.10, U2.11; no longer U$15.10, U7.11
- net LCD_RD: now also JP4.11, U2.12; no longer U$15.11, U7.12
- net LCD_WR: now also JP4.2, U2.44; no longer U$15.2, U7.44
- net LDO: now also C11.2; no longer C10.2
- net N$1: now also L3.2, U3.2; no longer L1.2, U2.2
- net N$10: now also U5.3; no longer U3.3
- net N$11: now also U5.6; no longer U3.6
- net N$12: now also U5.29; no longer U3.29
- net N$13: now also U5.7; no longer U3.7
- net N$14: now also U5.1; no longer U3.1
- net N$15: now also R1.1; no longer R5.1
- net N$16: now also U5.20; no longer U3.20
- net N$17: now also U5.24; no longer U3.24
- net N$18: now also R3.1; no longer R6.1
- net N$19: now also U5.30; no longer U3.30
- net N$2: now also L3.1, U3.4; no longer L1.1, U2.4
- net N$20: now also U5.2; no longer U3.2
- net N$21: now also U5.23; no longer U3.23
- net N$22: now also C37.2, U5.9; no longer C13.2, U3.9
- net N$23: now also R21.1, U5.25; no longer R4.1, U3.25
- net N$24: now also R22.1, U5.26; no longer R7.1, U3.26
- net N$25: now also R19.2, U5.28; no longer R8.2, U3.28
- net N$26: now also R16.1, R19.1; no longer R8.1, R9.1
- net N$27: now also C10.1, C14.1, C9.2, JP4.27; no longer C21.2, C22.1, C23.1, U$15.27
- net N$28: now also C44.1, U7.4; no longer C18.1, U6.4
- net N$29: now also C43.1, U7.1; no longer C17.1, U6.1
- net N$3: now also C19.1; no longer C5.1
- net N$32: now also U7.9; no longer U6.9
- net N$33: now also C9.1, JP4.26; no longer C21.1, U$15.26
- net N$34: now also C10.2, JP4.28; no longer C22.2, U$15.28
- net N$35: now also C14.2, JP4.29; no longer C23.2, U$15.29
- net N$36: now also C16.1, C17.2, C18.1, JP4.24; no longer C24.2, C25.1, C26.1, U$15.24
- net N$37: now also C17.1, JP4.25; no longer C24.1, U$15.25
- net N$38: now also C16.2, JP4.23; no longer C25.2, U$15.23
- net N$39: now also C18.2, JP4.22; no longer C26.2, U$15.22
- net N$4: now also U5.16, U5.17; no longer U3.16, U3.17
- net N$40: now also C2.1, JP4.31; no longer C28.1, U$15.31
- net N$41: now also C5.1, JP4.32; no longer C29.1, U$15.32
- net N$42: now also C1.1, JP4.21, JP4.30; no longer C27.1, U$15.21, U$15.30
- net N$43: now also C8.1, JP4.33; no longer C30.1, U$15.33
- net N$44: now also C12.1, JP4.34; no longer C31.1, U$15.34
- net N$45: now also C15.1, JP4.35, JP4.36; no longer C32.1, U$15.35, U$15.36
- net N$46: now also C36.1, R14.1, R15.2, U2.40; no longer C40.1, R16.1, R17.2, U7.40
- net N$47: now also JP6.1, U2.36; no longer JP3.1, U7.36
- net N$48: now also C45.1, U6.2, U6.3; no longer C14.1, U5.2, U5.3
- net N$49: now also JP6.2, U2.25; no longer JP3.2, U7.25
- net N$5: now also C19.2, L1.1; no longer C5.2, L2.1
- net N$50: now also C23.1, L2.1, U2.34, U2.35; no longer C47.1, L4.1, U7.34, U7.35
- net N$51: now also JP4.17; no longer U$15.17
- net N$52: now also JP4.16; no longer U$15.16
- net N$53: now also C27.2, C30.1, L2.2, U2.18; no longer C45.1, C46.2, L4.2, U7.18
- net N$54: now also C40.2, C41.1, L4.1, U7.2, U7.8; no longer C15.1, C16.2, L3.1, U6.2, U6.8
- net N$55: now also JP5.3; no longer JP4.3
- net N$56: now also JP5.5; no longer JP4.5
- net N$57: now also JP5.4; no longer JP4.4
- net N$6: now also C20.1; no longer C8.1
- net N$8: now also D2.A, R9.2; no longer D3.A, R1.2
- net N$88: now also R5.1, R7.2, R8.2; no longer R11.1, R2.2, R3.2
- net N$9: now also C32.1, R8.1, U3.6; no longer C34.1, R3.1, U2.6
- net PWR_TACT: now also R5.2, U2.23; no longer R11.2, U7.23
- net SD_!CS!: now also U2.6; no longer U7.6
- net SD_CRD_DET: now also C3.2, R2.2, U2.27; no longer C39.2, R10.2, U7.27
- net SD_MISO: now also U2.7; no longer U7.7
- net SD_MOSI: now also U2.8; no longer U7.8
- net SD_SCLK: now also U2.10; no longer U7.10
- net SENS_SCL: now also R6.1, U2.20, U6.5, U7.7; no longer R21.1, U5.5, U6.7, U7.20
- net SENS_SDA: now also R11.1, U2.24, U7.6; no longer R20.1, U5.6, U7.24
- net STAT_LED: now also R4.2; no longer R23.2
- net USB_D+: now also JP3.3, U2.16; no longer J1.3, U7.16
- net USB_D-: now also JP3.2, U2.15; no longer J1.2, U7.15
- net VBUS: now also C7.2, JP3.1, R9.1; no longer C9.2, J1.1, R1.1
- net VSYS: now also C25.1, C28.1, C31.1, C33.1, C38.2, L1.2, R1.2, R14.2, R3.2, U3.5, U3.7, U5.8; no longer C1.1, C12.2, C2.1, C6.1, C7.1, L2.2, R16.2, R5.2, R6.2, U2.5, U2.7, U3.8
- net V_BATT: now also C22.2; no longer C11.2

Commit message: Finished BOM
Parts:
- L1: value 1uH -> 1.2uH
- U2: value ATUCL4U-TQFP48 -> ATUC128L4U-TQFP48
Changed lines of the file:
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@@
 <layer number="47" name="Measures" color="7" fill="1" visible="no" active="yes"/>
 <layer number="48" name="Document" color="7" fill="1" visible="no" active="yes"/>
-<layer number="49" name="Reference" color="7" fill="1" visible="yes" active="yes"/>
+<layer number="49" name="Reference" color="7" fill="1" visible="no" active="yes"/>
 <layer number="50" name="dxf" color="7" fill="1" visible="no" active="no"/>
 <layer number="51" name="tDocu" color="6" fill="1" visible="yes" active="yes"/>
@@
 <elements>
 <element name="L3" library="hybridpi" package="SRU5028" value="2.2uH" x="21.65" y="105.25" rot="R270"/>
-<element name="L1" library="hybridpi" package="SRU5028" value="1uH" x="18" y="122" rot="R90"/>
-<element name="U1" library="hybridpi" package="VQFN-24" value="BQ24251" x="19" y="116" rot="R180"/>
+<element name="L1" library="hybridpi" package="SRU5028" value="1.2uH" x="18" y="122" rot="R90"/>
+<element name="U1" library="hybridpi" package="VQFN-24" value="BQ24251" x="19" y="116" rot="R180">
+<attribute name="VENDOR" value="DIGI-KEY" x="19" y="116" size="1.778" layer="27" rot="R180" display="off"/>
+<attribute name="VENDOR_PN" value="296-36444-1-ND" x="19" y="116" size="1.778" layer="27" rot="R180" display="off"/>
+</element>
 <element name="U3" library="hybridpi" package="WSON-12" value="LM3668-3034" x="16.25" y="107" rot="R90">
 <attribute name="EAGLEUP" value="WSON-12-3p1x3p1" x="16.25" y="107" size="1.778" layer="27" rot="R90" display="off"/>
+<attribute name="VENDOR" value="DIGI-KEY" x="16.25" y="107" size="1.778" layer="27" rot="R90" display="off"/>
+<attribute name="VENDOR_PN" value="LM3668SD-3034/NOPBCT-ND" x="16.25" y="107" size="1.778" layer="27" rot="R90" display="off"/>
 </element>
 <element name="C31" library="hybridpi-rcl" package="C0805" value="10uF" x="23" y="110">
@@
 <element name="D1" library="hybridpi-opto" package="LED-2-1.6X1.25" value="LED-RG-APT" x="2" y="121" rot="R90">
 <attribute name="EAGLEUP" value="LED-1p6x1p25" x="2" y="121" size="1.778" layer="27" rot="R90" display="off"/>
+<attribute name="VENDOR" value="DIGI-KEY" x="2" y="121" size="1.778" layer="27" rot="R90" display="off"/>
+<attribute name="VENDOR_PN" value="754-1146-1-ND" x="2" y="121" size="1.778" layer="27" rot="R90" display="off"/>
 </element>
 <element name="JP1" library="hybridpi-connector" package="JST-PH-2-RA" value="M02-JST-PH-2-RA" x="21" y="129" rot="R270">
 <attribute name="EAGLEUP" value="JST-PH-2-RA" x="21" y="129" size="1.778" layer="27" rot="R270" display="off"/>
+<attribute name="VENDOR" value="DIGI-KEY" x="21" y="129" size="1.778" layer="27" rot="R270" display="off"/>
+<attribute name="VENDOR_PN" value="455-1719-ND" x="21" y="129" size="1.778" layer="27" rot="R270" display="off"/>
 </element>
 <element name="C22" library="hybridpi-rcl" package="C0603" value="2.2uF" x="23.1" y="116.8" rot="R90">
@@
 <element name="U5" library="hybridpi-rf" package="UC530" value="UC530" x="36.25" y="7" rot="R270">
 <attribute name="EAGLEUP" value="UC530" x="36.25" y="7" size="1.778" layer="27" rot="R270" display="off"/>
+<attribute name="VENDOR" value="MOUSER" x="36.25" y="7" size="1.778" layer="27" rot="R270" display="off"/>
+<attribute name="VENDOR_PN" value="916-UC530" x="36.25" y="7" size="1.778" layer="27" rot="R270" display="off"/>
 </element>
 <element name="C38" library="hybridpi-rcl" package="C0603" value="1uF" x="28.5" y="7">
@@
 <element name="U6" library="hybridpi-sensor" package="BMP180" value="BMP180" x="4" y="41">
 <attribute name="EAGLEUP" value="BMP180" x="4" y="41" size="1.778" layer="27" display="off"/>
+<attribute name="VENDOR" value="DIGI-KEY" x="4" y="41" size="1.778" layer="27" display="off"/>
+<attribute name="VENDOR_PN" value="828-1027-1-ND" x="4" y="41" size="1.778" layer="27" display="off"/>
 </element>
 <element name="C45" library="hybridpi-rcl" package="C0603" value="0.1uF" x="4" y="45"/>
 <element name="U7" library="hybridpi-sensor" package="DFN-10-2X2" value="MAG3110" x="11" y="41" rot="R270">
 <attribute name="EAGLEUP" value="DFN-10-2x2" x="11" y="41" size="1.778" layer="27" rot="R270" display="off"/>
+<attribute name="VENDOR" value="DIGI-KEY" x="11" y="41" size="1.778" layer="27" rot="R270" display="off"/>
+<attribute name="VENDOR_PN" value="MAG3110FCR1CT-ND" x="11" y="41" size="1.778" layer="27" rot="R270" display="off"/>
 </element>
 <element name="C41" library="hybridpi-rcl" package="C0603" value="0.1uF" x="11" y="44" rot="R180"/>
@@
 <element name="JP2" library="hybridpi-connector" package="MICROSD-5031821853" value="MICRO-SD-5031821853" x="2" y="50" rot="R90">
 <attribute name="EAGLEUP" value="MICROSD-5031821853" x="2" y="50" size="1.778" layer="27" rot="R90" display="off"/>
+<attribute name="VENDOR" value="DIGI-KEY" x="2" y="50" size="1.778" layer="27" rot="R90" display="off"/>
+<attribute name="VENDOR_PN" value="WM9750CT-ND" x="2" y="50" size="1.778" layer="27" rot="R90" display="off"/>
 </element>
 <element name="C13" library="hybridpi-rcl" package="C0805" value="10uF" x="17.5" y="59" rot="R270">
@@
 <element name="JP4" library="hybridpi-connector" package="128240D" value="128240D" x="22" y="89" rot="R90">
 <attribute name="EAGLEUP" value="128240D_CON" x="22" y="89" size="1.778" layer="27" rot="R90" display="off"/>
+<attribute name="VENDOR" value="MOUSER" x="22" y="89" size="1.778" layer="27" rot="R90" display="off"/>
+<attribute name="VENDOR_PN" value="758-SEA8056-36" x="22" y="89" size="1.778" layer="27" rot="R90" display="off"/>
 </element>
 <element name="C9" library="hybridpi-rcl" package="C0603" value="1uF" x="17.5" y="93.9" rot="R90">
@@
 <attribute name="VENDOR_PN" value="587-1248-1-ND" x="50.75" y="4.95" size="1.778" layer="27" display="off"/>
 </element>
-<element name="U2" library="hybridpi-digitalic" package="TQFP48" value="ATUCL4U-TQFP48" x="14" y="82" rot="R180">
-<attribute name="EAGLEUP" value="TQFP-48" x="14" y="82" size="1.778" layer="27" rot="R180" display="off"/>
+<element name="U2" library="hybridpi-digitalic" package="TQFP48" value="ATUC128L4U-TQFP48" x="14" y="82" rot="R180">
+<attribute name="VENDOR" value="DIGI-KEY" x="14" y="82" size="1.778" layer="27" rot="R180" display="off"/>
+<attribute name="VENDOR_PN" value="ATUC128L4U-AUT-ND " x="14" y="82" size="1.778" layer="27" rot="R180" display="off"/>
 </element>
 <element name="R17" library="hybridpi-rcl" package="R0603" value="100K" x="5" y="71" rot="R180"/>
@@
 <element name="JP6" library="hybridpi-connector" package="JST-PH-2-RA" value="M02-JST-PH-2-RA" x="21" y="59" rot="R270">
 <attribute name="EAGLEUP" value="JST-PH-2-RA" x="21" y="59" size="1.778" layer="27" rot="R270" display="off"/>
+<attribute name="VENDOR" value="DIGI-KEY" x="21" y="59" size="1.778" layer="27" rot="R270" display="off"/>
+<attribute name="VENDOR_PN" value="455-1719-ND" x="21" y="59" size="1.778" layer="27" rot="R270" display="off"/>
 </element>
 <element name="S1" library="hybridpi-electromechanical" package="FSMRA" value="FSMRA7JH" x="14.45" y="130.75" rot="R180">
